File: Hardware/Simple_powerbank.kicad_sch (KiCad schematic)
At the start: 58 parts, among them IC1 MP2722GRH-0000-Z, J2 USB_C_Receptacle_USB2.0_16P, J3 Programming, Q2 NMOS, Q3 NMOS, SW1 Reset_button, U1 AP9101CK6, U2 ATtiny404-SS, U4 SRV05-4

Commit message: Zmieniono wartości kondensatorów
Parts:
- C13: value 2.2u -> 22u
- C7, C8: value 100n -> 220n
- C9: value 4.7u -> 220n
Changed lines of the file:
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@@
 			)
 		)
-		(property "Value" "100n"
+		(property "Value" "220n"
 			(at 267.97 34.2899 0)
 			(effects
@@
 			)
 		)
-		(property "Value" "100n"
+		(property "Value" "220n"
 			(at 205.74 148.5899 0)
 			(effects
@@
 			)
 		)
-		(property "Value" "2.2u"
+		(property "Value" "22u"
 			(at 151.13 33.0199 0)
 			(effects
@@
 			)
 		)
-		(property "Value" "4.7u"
+		(property "Value" "220n"
 			(at 74.93 81.2799 0)
 			(effects
