File: Hardware/Simple_powerbank.kicad_sch (KiCad schematic)
At the start: 58 parts, among them IC1 MP2722GRH-0000-Z, J2 USB_C_Receptacle_USB2.0_16P, J3 Programming, Q2 NMOS, Q3 NMOS, SW1 Reset_button, U1 AP9101CK6, U2 ATtiny404-SS, U4 SRV05-4

Commit message: Working sample
Parts:
- C17, C18: value 220n -> 470n
- C9: value 220n -> 4.7u
- D4: value LED -> Problem_led
- D5: value Problem_led -> Led
- R13: value 1k -> 1k5
Other:
- note added: "VCC filtering and bulk for ATTINY404 Place 4.7u near VCC Place 470n near ATTINY"
- note removed: "VCC filtering and bulk for ATTINY404 Place 4.7u near VCC Place 220n near ATTINY"
Changed lines of the file:
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@@
 		)
 	)
-	(text "VCC filtering and bulk for ATTINY404\nPlace 4.7u near VCC\nPlace 220n near ATTINY \n"
+	(text "VCC filtering and bulk for ATTINY404\nPlace 4.7u near VCC\nPlace 470n near ATTINY \n"
 		(exclude_from_sim no)
 		(at 86.36 71.12 0)
@@
 			)
 		)
-		(property "Value" "LED"
+		(property "Value" "Problem_led"
 			(at 181.2925 66.04 0)
 			(effects
@@
 			)
 		)
-		(property "Datasheet" "https://ngspice.sourceforge.io/docs/ngspice-html-manual/manual.xhtml#cha_MOSFETs"
+		(property "Datasheet" "https://www.tme.eu/pl/details/wms15n03t1-cyg/tranzystory-z-kanalem-n-smd/wayon/wms15n03t1/"
 			(at 85.09 27.94 0)
 			(effects
@@
 			)
 		)
-		(property "Value" "220n"
+		(property "Value" "470n"
 			(at 88.9 81.2799 0)
 			(effects
@@
 			)
 		)
-		(property "Value" "1k"
+		(property "Value" "1k5"
 			(at 190.5 66.04 90)
 			(effects
@@
 			)
 		)
-		(property "Datasheet" "https://www.way-on.cn/upload/202301/31/202301311441465755.pdf"
+		(property "Datasheet" "https://www.tme.eu/pl/details/wms15n03t1-cyg/tranzystory-z-kanalem-n-smd/wayon/wms15n03t1/"
 			(at 85.09 63.5 0)
 			(effects
@@
 			)
 		)
-		(property "Value" "Problem_led"
+		(property "Value" "Led"
 			(at 181.2925 57.15 0)
 			(effects
@@
 			)
 		)
-		(property "Value" "220n"
+		(property "Value" "4.7u"
 			(at 74.93 81.2799 0)
 			(effects
@@
 			)
 		)
-		(property "Value" "220n"
+		(property "Value" "470n"
 			(at 104.14 81.2799 0)
 			(effects
